File: kicad/tech_pcb.kicad_sch (KiCad schematic)
At the start: 24 parts, among them J1 Conn_01x10, J2 Conn_01x10, J3 USB_C_Receptacle_USB2.0_16P, J4 Conn_01x03_MountingPin, SW1 SW_Push, SW2 SW_Push, U1 STM32C071GBUxN, U2 XC6206PxxxMR

Commit message: Update part selections and add BOM
Parts:
- SW1, SW2: footprint Button_Switch_SMD:SW_SPST_TS-1088-xR025 -> Button_Switch_SMD:SW_Push_1P1T_NO_CK_KMR2
Changed lines of the file:
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@@
 			)
 		)
-		(property "Footprint" "Button_Switch_SMD:SW_SPST_TS-1088-xR025"
+		(property "Footprint" "Button_Switch_SMD:SW_Push_1P1T_NO_CK_KMR2"
 			(at 133.35 101.6 0)
 			(hide yes)
@@
 			)
 		)
-		(property "Footprint" "Button_Switch_SMD:SW_SPST_TS-1088-xR025"
+		(property "Footprint" "Button_Switch_SMD:SW_Push_1P1T_NO_CK_KMR2"
 			(at 125.73 119.38 0)
 			(hide yes)

Commit message: Update board to v0.2
Parts:
- removed J1, J2: Conn_01x10, Connector_PinHeader_2.54mm:PinHeader_1x10_P2.54mm_Vertical, symbol Connector_Generic:Conn_01x10
- added J1, J2: Conn_01x11, Connector_PinHeader_2.54mm:PinHeader_1x11_P2.54mm_Vertical, symbol Connector_Generic:Conn_01x11
- C3, C4: footprint Capacitor_SMD:C_0603_1608Metric -> Capacitor_SMD:C_0805_2012Metric
- D1, D2: footprint LED_SMD:LED_0603_1608Metric -> LED_SMD:LED_0805_2012Metric
- R3, R4, R5, R6: footprint Resistor_SMD:R_0603_1608Metric -> Resistor_SMD:R_0805_2012Metric
- SW1: value SW_Push -> RST
- SW2: value SW_Push -> BOOT
Connections:
- net PA2 is gone; now on net STATUS: U1.8 (PA2)
- net +3V3: now also J2.2 (Pin_2)
- net +5V: now also J2.1 (Pin_1)
- net GND: now also J1.3 (Pin_3), J2.3 (Pin_3)
- net NRST: now also J1.11 (Pin_11)
- net PA15: now also J1.1 (Pin_1)
- net PA3: now also J2.11 (Pin_11)
- net PA4: now also J2.10 (Pin_10)
- net PA5: now also J2.9 (Pin_9)
- net PA6: now also J2.8 (Pin_8)
- net PA7: now also J2.7 (Pin_7)
- net PA8: now also J2.4 (Pin_4)
- net PB0: now also J2.6 (Pin_6)
- net PB1: now also J2.5 (Pin_5)
- net PB3: now also J1.2 (Pin_2)
- net PB6: now also J1.6 (Pin_6)
- net PB7: now also J1.7 (Pin_7)
- net PB8: now also J1.8 (Pin_8)
- net STATUS: no longer U1.6 (PA0)
- net PC15: now reaches U1.1 (PC14)
- net PC15: now also J1.9 (Pin_9)
- net PC14: now reaches U1.2 (PC15)
- net PC14: now also J1.10 (Pin_10)
- net PB4: now reaches U1.24 (PB4)
- net PB4: now also J1.4 (Pin_4)
- net PB5: now reaches U1.25 (PB5)
- net PB5: now also J1.5 (Pin_5)
- net PA1: no longer names the net of U1.7 (PA1)
- no-connect marks 6 -> 4

Commit message: Tidy up the schematic
Parts:
- J1, J2: value Conn_01x11 -> 0.1" Pitch
- J4: value Conn_01x03_MountingPin -> SWD Header
- TP1: value TestPoint -> 3v3
- TP2: value TestPoint -> GND
- TP3: value TestPoint -> VBus
- TP4: value TestPoint -> Status
Connections:
- net +3V3: now also SW2.1; no longer SW2.2
- net BOOT0: now also SW2.2; no longer SW2.1
Other:
- note added: "Microcontroller"
- note added: "Pin Headers"
- note added: "Power Regulation"
- note added: "USB-C"
- company: (none) -> Tennessee Technological University
- title: (none) -> TN Tech PCB Design Workshop
- moved on the sheet: C1, C2, C3, C4, D1, D2, J1, J2, J3, J4, R1, R2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
